Commit message: add joint angle editor demo

File: examples/mycobot/mycobot.urdf (robot description, URDF)
Before this commit: robot firefighter, 10 links, 9 joints
Joints:
- removed joint joint6output_to_pump_head
- added joint camera_flange_to_pump_head: type fixed, parent camera_flange, child pump_head, origin xyz=0 0.016 0 rpy=0 0 0
- joint joint6output_to_camera_flange: origin xyz=0 0 0.01 rpy=1.579 0 0 -> xyz=0 0 0.01 rpy=1.5708 0 -2.3562
